File: kicad/_autosave-elote42.kicad_sch (KiCad schematic)
At the start: 86 parts, among them SW1 SW_Push, U1 ProMicro

Commit message: Placed components on PCB
Connections:
- net col5: no longer MX39.1 (COL)
- net at D39.2 (A): no longer MX39.2 (ROW)
Other:
- moved on the sheet: MX39
Changed lines of the file:
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@@
     (pin "2")
   )
-  (symbol (lib_id "MX_Alps_Hybrid:MX-NoLED") (at 138.43 115.57 0) (unit 1)
+  (symbol (lib_id "MX_Alps_Hybrid:MX-NoLED") (at 138.43 115.57 90) (unit 1)
     (in_bom yes) (on_board yes) (fields_autoplaced)
-    (property "Reference" "MX39" (id 0) (at 139.3156 109.22 0)
-      (effects (font (size 1.524 1.524)))
+    (property "Reference" "MX39" (id 0) (at 134.62 114.0494 90)
+      (effects (font (size 1.524 1.524)) (justify left))
     )
-    (property "Value" "MX-NoLED" (id 1) (at 139.3156 110.49 0)
-      (effects (font (size 0.508 0.508)))
+    (property "Value" "MX-NoLED" (id 1) (at 134.62 116.5893 90)
+      (effects (font (size 0.508 0.508)) (justify left))
     )
-    (property "Footprint" "MX_Alps_Hybrid:MX-1U-NoLED" (id 2) (at 122.555 116.205 0)
+    (property "Footprint" "MX_Alps_Hybrid:MX-1U-NoLED" (id 2) (at 139.065 131.445 0)
       (effects (font (size 1.524 1.524)) hide)
     )
-    (property "Datasheet" "" (id 3) (at 122.555 116.205 0)
+    (property "Datasheet" "" (id 3) (at 139.065 131.445 0)
       (effects (font (size 1.524 1.524)) hide)
     )
