File: kicad/elote42.kicad_pcb (KiCad board)
At the start: 2 copper layers, 318.3 x 95.2 mm, 86 parts, among them SW1 SW_Push, U1 ProMicro

Commit message: Moved pads closer to MCU
Parts:
- moved D15 8.73 mm to (40.5, 60.3)
- moved D16 8.73 mm to (59.5, 57.9)
- moved D17 8.73 mm to (78.6, 60.3)
- moved D27 8.73 mm to (40.5, 79.4)
- moved D28 8.73 mm to (59.5, 77.0)
- moved D29 8.73 mm to (78.6, 79.4)
- moved D3 8.73 mm to (40.5, 41.3)
- moved D37 8.73 mm to (69.1, 101.6)
- moved D39 8.73 mm to (112.7, 109.5)
- moved D4 8.73 mm to (59.5, 38.9)
- moved D5 8.73 mm to (78.6, 41.3)
- moved MX15 8.73 mm to (40.5, 54.8)
- moved MX16 8.73 mm to (59.5, 52.4)
- moved MX17 8.73 mm to (78.6, 54.8)
- moved MX27 8.73 mm to (40.5, 73.8)
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Other:
- board size 318.3 x 95.2 mm -> 322.3 x 95.2 mm

Commit message: tilted pads 10 degrees and tightened distance to mcu
Parts:
- moved SW1 46.5 mm to (149.2, 76.2)
- moved MX6 34.9 mm to (125.6, 58.2), turned to -10 degrees
- moved D6 33.5 mm to (124.0, 63.5), turned to -10 degrees
- moved MX5 33.2 mm to (107.2, 52.6), turned to -10 degrees
- moved MX4 32.3 mm to (88.9, 46.9), turned to -10 degrees
- moved MX18 32.1 mm to (122.2, 77.0), turned to -10 degrees
- moved MX7 32.0 mm to (172.7, 58.2), turned to 10 degrees
- moved D5 31.9 mm to (105.8, 57.9), turned to -10 degrees
- moved D7 31.4 mm to (173.6, 64.1), turned to 10 degrees
- moved MX3 31.4 mm to (69.3, 48.3), turned to -10 degrees
- moved D18 30.9 mm to (120.7, 82.5), turned to -10 degrees
- moved D4 30.9 mm to (87.3, 52.4), turned to -10 degrees
- moved MX17 30.2 mm to (103.9, 71.3), turned to -10 degrees
- moved MX2 30.1 mm to (49.3, 52.0), turned to -10 degrees
- moved MX8 30.1 mm to (191.0, 52.6), turned to 10 degrees
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Other:
- board size 322.3 x 95.2 mm -> 273.1 x 107.2 mm

Commit message: Routed columns on left and right pads
Routing:
- net col5: track 0.00 -> 76.9 mm
- net col6: track 0.00 -> 76.8 mm
- net col4: track 0.00 -> 71.3 mm
- net col3: track 0.00 -> 69.9 mm
- net col7: track 0.00 -> 69.4 mm
- net col8: track 0.00 -> 68.7 mm
- net col9: track 0.00 -> 41.8 mm
- net colA: track 0.00 -> 41.5 mm
- net colB: track 0.00 -> 41.5 mm
- net col0: track 0.00 -> 40.4 mm
- net col1: track 0.00 -> 40.3 mm
- net col2: track 0.00 -> 40.3 mm

Commit message: Routed diodes to corresponding switches
Parts:
- moved SW1 6.35 mm to (149.2, 82.5)
Routing:
- net Net-(D13-Pad2): track 0.00 -> 14.4 mm
- net Net-(D6-Pad2): track 0.00 -> 14.0 mm
- net Net-(D1-Pad2): track 0.00 -> 14.0 mm
- net Net-(D18-Pad2): track 0.00 -> 14.0 mm
- net Net-(D29-Pad2): track 0.00 -> 14.0 mm
- net Net-(D25-Pad2): track 0.00 -> 13.9 mm
- net Net-(D4-Pad2): track 0.00 -> 13.9 mm
- net Net-(D27-Pad2): track 0.00 -> 13.8 mm
- net Net-(D40-Pad2): track 0.00 -> 13.8 mm
- net Net-(D37-Pad2): track 0.00 -> 13.8 mm
- net Net-(D2-Pad2): track 0.00 -> 13.8 mm
- net Net-(D5-Pad2): track 0.00 -> 13.7 mm
- net Net-(D26-Pad2): track 0.00 -> 13.7 mm
- net Net-(D28-Pad2): track 0.00 -> 13.6 mm
- net Net-(D39-Pad2): track 0.00 -> 13.6 mm
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
Commit message: flipped diodes on right side for easier routing
Parts:
- moved SW1 2.38 mm to (149.2, 84.9)
- turned D10 to -170 degrees
- turned D11 to -170 degrees
- turned D12 to -170 degrees
- turned D19 to -170 degrees
- turned D20 to -170 degrees
- turned D21 to -170 degrees
- turned D22 to -170 degrees
- turned D23 to -170 degrees
- turned D24 to -170 degrees
- turned D31 to -170 degrees
- turned D32 to -170 degrees
- turned D33 to -170 degrees
- turned D34 to -170 degrees
- turned D35 to -170 degrees
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Connections:
- D12 pad 2: unconnected-(D12-Pad2) -> Net-(MX12-Pad2)
- D39 pad 2: Net-(D39-Pad2) -> unconnected-(D39-Pad2)
- MX12 pad 2: unconnected-(MX12-Pad2) -> Net-(MX12-Pad2)
- MX39 pad 1: col5 -> unconnected-(MX39-Pad1)
- MX39 pad 2: Net-(D39-Pad2) -> unconnected-(MX39-Pad2)
Routing:
- net Net-(D15-Pad2): track 0.00 -> 14.1 mm
- net Net-(D17-Pad2): track 0.00 -> 14.0 mm
- net Net-(D14-Pad2): track 0.00 -> 13.8 mm
- net Net-(D16-Pad2): track 0.00 -> 13.7 mm
- net unconnected-(D39-Pad2): track 0.00 -> 13.6 mm
- net Net-(D39-Pad2): track 13.6 -> 0.00 mm
- net Net-(D21-Pad2): track 0.00 -> 11.8 mm
- net Net-(D23-Pad2): track 0.00 -> 11.5 mm
- net Net-(D19-Pad2): track 0.00 -> 11.3 mm
- net Net-(MX12-Pad2): track 0.00 -> 11.3 mm
- net Net-(D20-Pad2): track 0.00 -> 11.1 mm
- net Net-(D22-Pad2): track 0.00 -> 10.7 mm
- net col9: track 41.8 -> 47.9 mm
- net col8: track 68.7 -> 74.0 mm
- net colB: track 41.5 -> 45.5 mm
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